File: PCB_ControladorMotor/PCB_CM/PCB_CM.kicad_sch (KiCad schematic)
At the start: 25 parts, among them J1 Conn_01x02_Socket, J2 Conn_01x02_Socket, J3 Conn_01x02_Socket, J4 Conn_01x02_Socket, Q1 IRF540N, U1 LM324A, U2 ATtiny85V-10P

Commit message: Add files via upload
Connections:
- net at H4.1, J3.2 (Pin_2), R4.2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: now also R7.2, U2.7 (PB2)
